File: qgpio.kicad_pcb (KiCad board)
At the start: 2 copper layers, 25.4 x 24.1 mm, 25 parts, among them J1 I2C_STANDARDQWIIC, J2 I2C_STANDARDQWIIC, J3 Conn_02x10_Odd_Even, U1 PCF8574A

Commit message: added I2C addr to back silk
Parts:
- moved LOGO1 0.63 mm to (160.0, 105.4)
Other:
- board text added: "A0111"
- board text added: "A6-3"
- board text added: "_0100"
Changed lines of the file:
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@@
   (general
     (thickness 1.6)
-    (drawings 46)
+    (drawings 49)
     (tracks 161)
     (zones 0)
@@
   (page A4)
   (layers
-    (0 F.Cu signal)
-    (31 B.Cu signal hide)
+    (0 F.Cu signal hide)
+    (31 B.Cu signal)
     (32 B.Adhes user hide)
     (33 F.Adhes user hide)
-    (34 B.Paste user hide)
-    (35 F.Paste user)
-    (36 B.SilkS user hide)
-    (37 F.SilkS user)
-    (38 B.Mask user hide)
-    (39 F.Mask user)
+    (34 B.Paste user)
+    (35 F.Paste user hide)
+    (36 B.SilkS user)
+    (37 F.SilkS user hide)
+    (38 B.Mask user)
+    (39 F.Mask user hide)
     (40 Dwgs.User user hide)
     (41 Cmts.User user hide)
@@
     (44 Edge.Cuts user)
     (45 Margin user hide)
-    (46 B.CrtYd user hide)
-    (47 F.CrtYd user)
-    (48 B.Fab user hide)
-    (49 F.Fab user)
+    (46 B.CrtYd user)
+    (47 F.CrtYd user hide)
+    (48 B.Fab user)
+    (49 F.Fab user hide)
   )
   (setup
-    (last_trace_width 0.254)
+    (last_trace_width 0.1524)
     (user_trace_width 0.1524)
     (user_trace_width 0.254)
@@
       (effects (font (size 1 1) (thickness 0.15)))
     )
-    (fp_text user %R (at 0 0 90) (layer F.Fab)
-      (effects (font (size 0.4 0.4) (thickness 0.06)))
-    )
     (fp_line (start 1.2 0.6) (end -1.2 0.6) (layer F.CrtYd) (width 0.05))
     (fp_line (start 1.2 -0.6) (end 1.2 0.6) (layer F.CrtYd) (width 0.05))
@@
     (fp_line (start -0.8 -0.4) (end 0.8 -0.4) (layer F.Fab) (width 0.1))
     (fp_line (start -0.8 0.4) (end -0.8 -0.4) (layer F.Fab) (width 0.1))
+    (fp_text user %R (at 0 0 90) (layer F.Fab)
+      (effects (font (size 0.4 0.4) (thickness 0.06)))
+    )
     (pad 2 smd roundrect (at 0.7 0 270) (size 0.7 0.8) (layers F.Cu F.Paste F.Mask) (roundrect_rratio 0.25)
       (net 27 "Net-(D10-Pad2)"))
@@
     (fp_text value LED (at 0 1.43 90) (layer F.Fab)
       (effects (font (size 1 1) (thickness 0.15)))
-    )
-    (fp_text user %R (at 0 0 90) (layer F.Fab)
-      (effects (font (size 0.4 0.4) (thickness 0.06)))
     )
     (fp_line (start 0.8 -0.4) (end -0.5 -0.4) (layer F.Fab) (width 0.1))
@@
     (fp_line (start 0.2286 -0.3556) (end -0.2032 0) (layer F.SilkS) (width 0.12))
     (fp_line (start -0.2032 0) (end 0.2286 0.3556) (layer F.SilkS) (width 0.12))
+    (fp_text user %R (at 0 0 90) (layer F.Fab)
+      (effects (font (size 0.4 0.4) (thickness 0.06)))
+    )
     (pad 2 smd roundrect (at 0.7875 0 90) (size 0.875 0.95) (layers F.Cu F.Paste F.Mask) (roundrect_rratio 0.25)
       (net 27 "Net-(D10-Pad2)"))
@@
   )
   (module Symbol:OSHW-Logo2_7.3x6mm_SilkScreen (layer B.Cu)
-    (at 160.02 104.775 180)
+    (at 160.02 105.41 180)
     (descr "Open Source Hardware Symbol")
     (tags "Logo Symbol OSHW")
@@
     )
   )
+  (gr_text A0111 (at 160.02 100.965) (layer B.SilkS)
+    (effects (font (size 1.27 1.016) (thickness 0.1524)) (justify mirror))
+  )
+  (gr_text _0100 (at 160.02 99.06) (layer B.SilkS)
+    (effects (font (size 1.27 1.016) (thickness 0.1524)) (justify mirror))
+  )
+  (gr_text A6-3 (at 160.02 97.155) (layer B.SilkS)
+    (effects (font (size 1.27 1.016) (thickness 0.1524)) (justify mirror))
+  )
   (gr_arc (start 140.97 118.11) (end 140.97 119.126) (angle 180) (layer B.SilkS) (width 0.254))
   (gr_text PWR (at 161.925 103.632) (layer F.SilkS)
@@
     (effects (font (size 1.27 1.016) (thickness 0.1524)) (justify mirror))
   )
-  (gr_text PCF8574 (at 155.575 96.52) (layer B.SilkS)
+  (gr_text PCF8574 (at 146.05 96.52) (layer B.SilkS)
     (effects (font (size 1.27 1.016) (thickness 0.1524)) (justify mirror))
   )
